Commit message: x_ball_description: position lwa4p arm in the summit-x

File: x_ball_description/robots/x_ball.urdf.xacro (robot description, xacro)
@@ -55,4 +55,8 @@
 		<origin xyz="-${wheel_offset_x} -${wheel_offset_y} ${wheel_offset_z}" rpy="0 0 0"/>
 	</xacro:omni_wheel>
+	<!-- ARM -->
+ 	<xacro:schunk_lwa4p name="arm" parent="rover_link" has_podest="true">
+		<origin xyz="-0.1 0 0.19" rpy="0 0 0" />
+	</xacro:schunk_lwa4p>
 	<!-- SENSORS -->
 <!--
@@ -94,7 +98,3 @@
 	</xacro:sensor_fotonic>
 -->
-	<!-- arm -->
- 	<xacro:schunk_lwa4d name="arm" parent="rover_link" has_podest="true">
-		<origin xyz="0 0 0.026" rpy="0 0 0" /> <!--slightly above gazebo plane-->
-	</xacro:schunk_lwa4d>
 </robot>
