Commit message: x_ball_description: adding x_ball with pg70 gripper

File: x_ball_description/robots/x_ball_pg70.urdf.xacro (robot description, xacro)
@@ -15,4 +15,6 @@
 	<xacro:include filename="$(find schunk_description)/urdf/materials.urdf.xacro" />
 	<xacro:include filename="$(find schunk_description)/urdf/lwa4p/lwa4p.urdf.xacro" />
+	<!-- Import PG70 gripper -->
+	<xacro:include filename="$(find schunk_description)/urdf/pg70/pg70.urdf.xacro" />
 	<!-- ***************** -->
 	<!-- Global parameters -->
@@ -57,4 +59,8 @@
 		<origin xyz="-0.1 0 0.19" rpy="0 0 0" />
 	</xacro:schunk_lwa4p>
+	<!-- gripper -->
+	<xacro:schunk_pg70 name="pg70" parent="arm_6_link">
+		<origin xyz="0 0 0.075" rpy="0 0 0" />
+	</xacro:schunk_pg70>
 	<!-- SENSORS -->
 <!--
